Commit message: saftey-commit while building urdf

File: urdf/dynamic_ef.urdf.xacro (robot description, xacro)
@@ -3,12 +3,69 @@
   <xacro:property name="height" value="2.0" />
   <xacro:property name="pi" value="3.141592654" />
+  <material name="blue">
+    <color rgba="0 0 0.8 0.8"/>
+  </material>
   <link name="base_link">
     <visual>
       <origin xyz="0 0 0.09" rpy="${pi/2.0} 0 0" />
       <geometry>
-        <!-- <box size="${height*0.05} ${height*0.05} ${height*0.1}" /> -->
         <mesh filename="package://dynamic_end_effector/meshes/h54-200-s500-r.stl" scale="0.001 0.001 0.001"/>
-        <!-- <box size="1 2 3"/> -->
       </geometry>
+      <material name="blue"/>
+    </visual>
+    <collision>
+      <origin xyz="0 0 0.063"/>
+      <geometry>
+        <box size="0.055 0.055 0.126"/>
+      </geometry>
+    </collision>
+  </link>
+  <joint name="base_link_to_base_yaw_link_joint" type="continuous">
+    <parent link="base_link"/>
+    <child link="base_yaw_link"/>
+    <origin xyz="0 0 0.126"/>
+    <axis xyz="0 0 1"/>
+  </joint>
+  <link name="base_yaw_link">
+    <visual>
+      <origin xyz="0 0 0" rpy="0 0 0" />
+      <geometry>
+        <mesh filename="package://dynamic_end_effector/meshes/assembly_base.stl" scale="0.001 0.001 0.001"/>
+      </geometry>
+      <material name="blue"/>
+    </visual>
+    <inertial>
+      <mass value="10"/>
+      <inertia ixx="0.01" ixy="0.01" ixz="0.01" iyy="0.01" iyz="0.01" izz="0.01"/>
+    </inertial>
+  </link>
+  <joint name="base_yaw_link_to_first_link_joint" type="continuous">
+    <parent link="base_yaw_link"/>
+    <child link="first_link"/>
+    <origin xyz="0 0 0.042"/>
+    <axis xyz="1 0 0"/>
+  </joint>
+  <link name="first_link">
+    <visual>
+      <origin xyz="0 0 0" rpy="0 0 0" />
+      <geometry>
+        <mesh filename="package://dynamic_end_effector/meshes/assembly_linkOne.stl" scale="0.001 0.001 0.001"/>
+      </geometry>
+      <material name="blue"/>
+    </visual>
+  </link>
+  <joint name="first_link_to_second_link_joint" type="continuous">
+    <parent link="first_link"/>
+    <child link="second_link"/>
+    <origin xyz="0 0.806 0"/>
+    <axis xyz="1 0 0"/>
+  </joint>
+  <link name="second_link">
+    <visual>
+      <origin xyz="-0.033 0 0" rpy="0 ${pi/2.0} ${pi/2.0}" />
+      <geometry>
+        <mesh filename="package://dynamic_end_effector/meshes/assembly_linkTwo.stl" scale="0.001 0.001 0.001"/>
+      </geometry>
+      <material name="blue"/>
     </visual>
   </link>
