Commit message: hi

File: urdf/dynamic-ef.urdf.xacro (robot description, xacro)
@@ -1,6 +1,10 @@
 <?xml version="1.0"?>
 <robot name="dyn_ef_robot" xmlns:xacro="http://www.ros.org/wiki/xacro">
-  <xacro:property name="height" value="2.0" />
-  <!-- <xacro:property name="pi" value="3.141592654" /> -->
+  <gazebo>
+    <plugin name="gazebo_ros_control" filename="libgazebo_ros_control.so">
+      <robotNamespace>/dyn_ef_robot</robotNamespace>
+    </plugin>
+  </gazebo>
+  <xacro:property name="height" value="0.0" />
   <xacro:macro name="default_inertial" params="mass">
     <inertial>
@@ -9,7 +13,20 @@
     </inertial>
   </xacro:macro>
+  <xacro:macro name="transmission_block" params="joint_name">
+    <transmission name="trans_${joint_name}">
+      <type>transmission_interface/SimpleTransmission</type>
+      <joint name="${joint_name}">
+        <hardwareInterface>PositionJointInterface</hardwareInterface>
+      </joint>
+      <actuator name="motor_${joint_name}">
+        <hardwareInterface>PositionJointInterface</hardwareInterface>
+        <mechanicalReduction>1</mechanicalReduction>
+      </actuator>
+    </transmission>
+  </xacro:macro>
   <material name="blue">
     <color rgba="0 0 0.8 1"/>
   </material>
+  <!--                                start listing links and joints                                                -->
   <link name="world"/>
   <joint name="fixy" type="fixed">
@@ -37,5 +54,7 @@
     <origin xyz="0 0 0.126"/>
     <axis xyz="0 0 1"/>
+    <dynamics damping="1.0" friction="5.0"/>
   </joint>
+  <xacro:transmission_block joint_name="base_link_to_base_yaw_link_joint"/>
   <link name="base_yaw_link">
     <visual>
@@ -62,7 +81,8 @@
     <origin xyz="0 0 0.042"/>
     <axis xyz="1 0 0"/>
-    <dynamics damping="1.0" friction="5.0"/>
+    <dynamics damping="1.0" friction="1.0"/>
     <limit upper="2.0" lower="-2.0" effort="45" velocity="1"/>
   </joint>
+  <xacro:transmission_block joint_name="base_yaw_link_to_first_link_joint"/>
   <link name="first_link">
     <visual>
@@ -87,4 +107,5 @@
     <dynamics damping="1.0" friction="5.0"/>
   </joint>
+  <xacro:transmission_block joint_name="first_link_to_second_link_joint"/>
   <link name="second_link">
     <visual>
@@ -109,4 +130,5 @@
     <dynamics damping="1.0" friction="5.0"/>
   </joint>
+  <xacro:transmission_block joint_name="second_link_to_third_link_joint"/>
   <link name="third_link">
     <visual>
@@ -131,4 +153,5 @@
     <dynamics damping="1.0" friction="5.0"/>
   </joint>
+  <xacro:transmission_block joint_name="third_link_to_fourth_link_joint"/>
   <link name="fourth_link">
     <visual>
@@ -155,4 +178,5 @@
     <dynamics damping="1.0" friction="5.0"/>
   </joint>
+  <xacro:transmission_block joint_name="fourth_link_to_fifth_link_joint"/>
   <link name="fifth_link">
     <visual>

Commit message: added camera, improved joint limits, kind of fixed errors

File: urdf/dynamic-ef.urdf.xacro (robot description, xacro)
@@ -6,5 +6,9 @@
     </plugin>
   </gazebo>
+  <material name="red">
+    <color rgba="1.0 0 0 1.0"/>
+  </material>
   <xacro:property name="height" value="0.0" />
+  <xacro:property name="camera_link_size" value="0.05" /> <!-- Size of square 'camera' box -->
   <xacro:macro name="default_inertial" params="mass">
     <inertial>
@@ -17,8 +21,8 @@
       <type>transmission_interface/SimpleTransmission</type>
       <joint name="${joint_name}">
-        <hardwareInterface>PositionJointInterface</hardwareInterface>
+        <hardwareInterface>hardware_interface/PositionJointInterface</hardwareInterface>
       </joint>
       <actuator name="motor_${joint_name}">
-        <hardwareInterface>PositionJointInterface</hardwareInterface>
+        <hardwareInterface>hardware_interface/PositionJointInterface</hardwareInterface>
         <mechanicalReduction>1</mechanicalReduction>
       </actuator>
@@ -49,5 +53,5 @@
     <xacro:default_inertial mass="0.8"/>
   </link>
-  <joint name="base_link_to_base_yaw_link_joint" type="continuous">
+  <joint name="base_link_to_base_yaw_link_joint" type="revolute">
     <parent link="base_link"/>
     <child link="base_yaw_link"/>
@@ -55,4 +59,5 @@
     <axis xyz="0 0 1"/>
     <dynamics damping="1.0" friction="5.0"/>
+    <limit upper="${pi}" lower="${-pi}" effort="45" velocity="1"/>
   </joint>
   <xacro:transmission_block joint_name="base_link_to_base_yaw_link_joint"/>
@@ -100,5 +105,5 @@
     <xacro:default_inertial mass="2"/>
   </link>
-  <joint name="first_link_to_second_link_joint" type="continuous">
+  <joint name="first_link_to_second_link_joint" type="revolute">
     <parent link="first_link"/>
     <child link="second_link"/>
@@ -106,4 +111,5 @@
     <axis xyz="1 0 0"/>
     <dynamics damping="1.0" friction="5.0"/>
+    <limit upper="${0.9*pi}" lower="${-0.9*pi}" effort="45" velocity="1"/>
   </joint>
   <xacro:transmission_block joint_name="first_link_to_second_link_joint"/>
@@ -129,4 +135,5 @@
     <axis xyz="0 0 1"/>
     <dynamics damping="1.0" friction="5.0"/>
+    <limit upper="${pi}" lower="${-pi}" effort="45" velocity="1"/>
   </joint>
   <xacro:transmission_block joint_name="second_link_to_third_link_joint"/>
@@ -152,4 +159,5 @@
     <axis xyz="1 0 0"/>
     <dynamics damping="1.0" friction="5.0"/>
+    <limit upper="2.0" lower="-2.0" effort="45" velocity="1"/>
   </joint>
   <xacro:transmission_block joint_name="third_link_to_fourth_link_joint"/>
@@ -171,5 +179,5 @@
     <xacro:default_inertial mass="0.3"/>
   </link>
-  <joint name="fourth_link_to_fifth_link_joint" type="continuous">
+  <joint name="fourth_link_to_fifth_link_joint" type="revolute">
     <parent link="fourth_link"/>
     <child link="fifth_link"/>
@@ -177,4 +185,5 @@
     <axis xyz="0 0 1"/>
     <dynamics damping="1.0" friction="5.0"/>
+    <limit upper="${pi}" lower="${-pi}" effort="45" velocity="1"/>
   </joint>
   <xacro:transmission_block joint_name="fourth_link_to_fifth_link_joint"/>
@@ -196,3 +205,76 @@
     <xacro:default_inertial mass="0.01"/>
   </link>
+  <joint name="camera_joint" type="fixed">
+    <!-- <axis xyz="0 1 0" /> -->
+    <origin xyz="0 0 ${camera_link_size/2 + 0.01}" rpy="0 0 0"/>
+    <parent link="fifth_link"/>
+    <child link="camera_link"/>
+  </joint>
+  <!-- Camera -->
+  <link name="camera_link">
+    <collision>
+      <origin xyz="0 0 0" rpy="0 0 0"/>
+      <geometry>
+        <box size="${camera_link_size} ${camera_link_size} ${camera_link_size}"/>
+      </geometry>
+    </collision>
+    <visual>
+      <origin xyz="0 0 0" rpy="0 0 0"/>
+      <geometry>
+        <box size="${camera_link_size} ${camera_link_size} ${camera_link_size}"/>
+      </geometry>
+    </visual>
+    <inertial>
+      <mass value="1e-5" />
+      <origin xyz="0 0 0" rpy="0 0 0"/>
+      <inertia ixx="1e-6" ixy="0" ixz="0" iyy="1e-6" iyz="0" izz="1e-6" />
+    </inertial>
+  </link>
+  <!-- <gazebo reference="camera_link">
+  </gazebo> -->
+    <!-- camera -->
+  <gazebo reference="camera_link">
+    <visual>
+      <material>
+        <ambient>0.70 0.19225 0.19225 1.0</ambient>
+        <diffuse>0.90 0.50754 0.50754 1.0</diffuse>
+        <specular>0.90 0.508273 0.508273 1.0</specular>
+        <emissive>0.0 0.0 0.0 0.0</emissive>
+      </material>
+    </visual>
+    <sensor type="camera" name="camera1">
+      <update_rate>30.0</update_rate>
+      <camera name="head">
+        <horizontal_fov>1.3962634</horizontal_fov>
+        <image>
+          <width>800</width>
+          <height>800</height>
+          <format>R8G8B8</format>
+        </image>
+        <clip>
+          <near>0.02</near>
+          <far>300</far>
+        </clip>
+        <noise>
+          <type>gaussian</type>
+          <mean>0.0</mean>
+          <stddev>0.007</stddev>
+        </noise>
+      </camera>
+      <plugin name="camera_controller" filename="libgazebo_ros_camera.so">
+        <alwaysOn>true</alwaysOn>
+        <updateRate>0.0</updateRate>
+        <cameraName>dyn_ef_robot/camera1</cameraName>
+        <imageTopicName>image_raw</imageTopicName>
+        <cameraInfoTopicName>camera_info</cameraInfoTopicName>
+        <frameName>camera_link</frameName>
+        <hackBaseline>0.07</hackBaseline>
+        <distortionK1>0.0</distortionK1>
+        <distortionK2>0.0</distortionK2>
+        <distortionK3>0.0</distortionK3>
+        <distortionT1>0.0</distortionT1>
+        <distortionT2>0.0</distortionT2>
+      </plugin>
+    </sensor>
+  </gazebo>
 </robot>

Commit message: added 2nd file to store all gazebo things for the URDF

File: urdf/dynamic-ef.urdf.xacro (robot description, xacro)
@@ -1,14 +1,17 @@
 <?xml version="1.0"?>
 <robot name="dyn_ef_robot" xmlns:xacro="http://www.ros.org/wiki/xacro">
-  <gazebo>
-    <plugin name="gazebo_ros_control" filename="libgazebo_ros_control.so">
-      <robotNamespace>/dyn_ef_robot</robotNamespace>
-    </plugin>
-  </gazebo>
+  <!-- Import all Gazebo-customization elements, including Gazebo colors -->
+  <xacro:include filename="$(find dynamic_end_effector)/urdf/dynamic-ef.gazebo" />
+  <!-- RViz-only colors -->
   <material name="red">
     <color rgba="1.0 0 0 1.0"/>
   </material>
+  <material name="blue">
+    <color rgba="0 0 0.8 1"/>
+  </material>
+  <!-- some properties for the urdf file -->
   <xacro:property name="height" value="0.0" />
   <xacro:property name="camera_link_size" value="0.05" /> <!-- Size of square 'camera' box -->
+  <!-- inertias for all links -->
   <xacro:macro name="default_inertial" params="mass">
     <inertial>
@@ -17,4 +20,5 @@
     </inertial>
   </xacro:macro>
+  <!-- interface between moveit and gazebo controllers -->
   <xacro:macro name="transmission_block" params="joint_name">
     <transmission name="trans_${joint_name}">
@@ -29,8 +33,5 @@
     </transmission>
   </xacro:macro>
-  <material name="blue">
-    <color rgba="0 0 0.8 1"/>
-  </material>
-  <!--                                start listing links and joints                                                -->
+  <!--  ##################### start listing links and joints  ##############################  -->
   <link name="world"/>
   <joint name="fixy" type="fixed">
@@ -165,5 +166,4 @@
     <visual>
       <origin xyz="0 0 0" rpy="${pi/2.0} 0 ${pi/2.0}" />
-      <!-- <origin xyz="0 0 0" rpy="0 0 0"/> -->
       <geometry>
         <mesh filename="package://dynamic_end_effector/meshes/assembly_linkFour.stl" scale="0.001 0.001 0.001"/>
@@ -172,5 +172,4 @@
     <collision>
       <origin xyz="0 0 0" rpy="${pi/2.0} 0 ${pi/2.0}" />
-      <!-- <origin xyz="0 0 0" rpy="0 0 0"/> -->
       <geometry>
         <mesh filename="package://dynamic_end_effector/meshes/assembly_linkFour.stl" scale="0.001 0.001 0.001"/>
@@ -191,5 +190,4 @@
     <visual>
       <origin xyz="0 0 0" rpy="${pi/2.0} 0 0" />
-      <!-- <origin xyz="0 0 0" rpy="0 0 0"/> -->
       <geometry>
         <mesh filename="package://dynamic_end_effector/meshes/assembly_linkFive.stl" scale="0.001 0.001 0.001"/>
@@ -198,5 +196,4 @@
     <collision>
       <origin xyz="0 0 0" rpy="${pi/2.0} 0 0" />
-      <!-- <origin xyz="0 0 0" rpy="0 0 0"/> -->
       <geometry>
         <mesh filename="package://dynamic_end_effector/meshes/assembly_linkFive.stl" scale="0.001 0.001 0.001"/>
@@ -205,4 +202,5 @@
     <xacro:default_inertial mass="0.01"/>
   </link>
+  <!-- fixed camera joint -->
   <joint name="camera_joint" type="fixed">
     <!-- <axis xyz="0 1 0" /> -->
@@ -231,50 +229,3 @@
     </inertial>
   </link>
-  <!-- <gazebo reference="camera_link">
-  </gazebo> -->
-    <!-- camera -->
-  <gazebo reference="camera_link">
-    <visual>
-      <material>
-        <ambient>0.70 0.19225 0.19225 1.0</ambient>
-        <diffuse>0.90 0.50754 0.50754 1.0</diffuse>
-        <specular>0.90 0.508273 0.508273 1.0</specular>
-        <emissive>0.0 0.0 0.0 0.0</emissive>
-      </material>
-    </visual>
-    <sensor type="camera" name="camera1">
-      <update_rate>30.0</update_rate>
-      <camera name="head">
-        <horizontal_fov>1.3962634</horizontal_fov>
-        <image>
-          <width>800</width>
-          <height>800</height>
-          <format>R8G8B8</format>
-        </image>
-        <clip>
-          <near>0.02</near>
-          <far>300</far>
-        </clip>
-        <noise>
-          <type>gaussian</type>
-          <mean>0.0</mean>
-          <stddev>0.007</stddev>
-        </noise>
-      </camera>
-      <plugin name="camera_controller" filename="libgazebo_ros_camera.so">
-        <alwaysOn>true</alwaysOn>
-        <updateRate>0.0</updateRate>
-        <cameraName>dyn_ef_robot/camera1</cameraName>
-        <imageTopicName>image_raw</imageTopicName>
-        <cameraInfoTopicName>camera_info</cameraInfoTopicName>
-        <frameName>camera_link</frameName>
-        <hackBaseline>0.07</hackBaseline>
-        <distortionK1>0.0</distortionK1>
-        <distortionK2>0.0</distortionK2>
-        <distortionK3>0.0</distortionK3>
-        <distortionT1>0.0</distortionT1>
-        <distortionT2>0.0</distortionT2>
-      </plugin>
-    </sensor>
-  </gazebo>
 </robot>

Commit message: added apriltag-world to gazebo-simulation, changed rotation of camera link in urdf

File: urdf/dynamic-ef.urdf.xacro (robot description, xacro)
@@ -205,5 +205,5 @@
   <joint name="camera_joint" type="fixed">
     <!-- <axis xyz="0 1 0" /> -->
-    <origin xyz="0 0 ${camera_link_size/2 + 0.01}" rpy="0 0 0"/>
+    <origin xyz="0 0 ${camera_link_size/2 + 0.01}" rpy="0 ${-pi/2} 0"/>
     <parent link="fifth_link"/>
     <child link="camera_link"/>

Commit message: added safety-controller in urdf

File: urdf/dynamic-ef.urdf.xacro (robot description, xacro)
@@ -55,4 +55,5 @@
   </link>
   <joint name="base_link_to_base_yaw_link_joint" type="revolute">
+    <safety_controller k_position="100.0" k_velocity="40.0" soft_lower_limit="${-pi}" soft_upper_limit="${pi}"/>
     <parent link="base_link"/>
     <child link="base_yaw_link"/>
@@ -60,5 +61,5 @@
     <axis xyz="0 0 1"/>
     <dynamics damping="1.0" friction="5.0"/>
-    <limit upper="${pi}" lower="${-pi}" effort="45" velocity="1"/>
+    <limit upper="${pi}" lower="${-pi}" effort="45" velocity="5"/>
   </joint>
   <xacro:transmission_block joint_name="base_link_to_base_yaw_link_joint"/>
@@ -83,4 +84,5 @@
   </link>
   <joint name="base_yaw_link_to_first_link_joint" type="revolute">
+    <safety_controller k_position="100.0" k_velocity="40.0" soft_lower_limit="-2.0" soft_upper_limit="2.0"/>
     <parent link="base_yaw_link"/>
     <child link="first_link"/>
@@ -88,5 +90,5 @@
     <axis xyz="1 0 0"/>
     <dynamics damping="1.0" friction="1.0"/>
-    <limit upper="2.0" lower="-2.0" effort="45" velocity="1"/>
+    <limit upper="2.0" lower="-2.0" effort="45" velocity="5"/>
   </joint>
   <xacro:transmission_block joint_name="base_yaw_link_to_first_link_joint"/>
@@ -107,4 +109,5 @@
   </link>
   <joint name="first_link_to_second_link_joint" type="revolute">
+    <safety_controller k_position="100.0" k_velocity="40.0" soft_lower_limit="${-0.9*pi}" soft_upper_limit="${0.9*pi}"/>
     <parent link="first_link"/>
     <child link="second_link"/>
@@ -112,5 +115,5 @@
     <axis xyz="1 0 0"/>
     <dynamics damping="1.0" friction="5.0"/>
-    <limit upper="${0.9*pi}" lower="${-0.9*pi}" effort="45" velocity="1"/>
+    <limit upper="${0.9*pi}" lower="${-0.9*pi}" effort="45" velocity="5"/>
   </joint>
   <xacro:transmission_block joint_name="first_link_to_second_link_joint"/>
@@ -131,4 +134,5 @@
   </link>
   <joint name="second_link_to_third_link_joint" type="continuous">
+    <safety_controller k_position="100.0" k_velocity="40.0" soft_lower_limit="${-pi}" soft_upper_limit="${pi}"/>
     <parent link="second_link"/>
     <child link="third_link"/>
@@ -136,5 +140,5 @@
     <axis xyz="0 0 1"/>
     <dynamics damping="1.0" friction="5.0"/>
-    <limit upper="${pi}" lower="${-pi}" effort="45" velocity="1"/>
+    <limit upper="${pi}" lower="${-pi}" effort="45" velocity="5"/>
   </joint>
   <xacro:transmission_block joint_name="second_link_to_third_link_joint"/>
@@ -154,5 +158,6 @@
     <xacro:default_inertial mass="0.1"/>
   </link>
-  <joint name="third_link_to_fourth_link_joint" type="continuous">
+  <joint name="third_link_to_fourth_link_joint" type="revolute">
+    <safety_controller k_position="100.0" k_velocity="40.0" soft_lower_limit="-2.0" soft_upper_limit="2.0"/>
     <parent link="third_link"/>
     <child link="fourth_link"/>
@@ -160,5 +165,5 @@
     <axis xyz="1 0 0"/>
     <dynamics damping="1.0" friction="5.0"/>
-    <limit upper="2.0" lower="-2.0" effort="45" velocity="1"/>
+    <limit upper="2.0" lower="-2.0" effort="45" velocity="5"/>
   </joint>
   <xacro:transmission_block joint_name="third_link_to_fourth_link_joint"/>
@@ -179,4 +184,5 @@
   </link>
   <joint name="fourth_link_to_fifth_link_joint" type="revolute">
+    <safety_controller k_position="100.0" k_velocity="40.0" soft_lower_limit="${-pi}" soft_upper_limit="${pi}"/>
     <parent link="fourth_link"/>
     <child link="fifth_link"/>
@@ -184,5 +190,5 @@
     <axis xyz="0 0 1"/>
     <dynamics damping="1.0" friction="5.0"/>
-    <limit upper="${pi}" lower="${-pi}" effort="45" velocity="1"/>
+    <limit upper="${pi}" lower="${-pi}" effort="45" velocity="5"/>
   </joint>
   <xacro:transmission_block joint_name="fourth_link_to_fifth_link_joint"/>
