Commit message: urdf updated to new design, meshes added

File: urdf/dynamic-ef.urdf.xacro (robot description, xacro)
@@ -12,5 +12,5 @@
   <!-- some properties for the urdf file -->
   <xacro:property name="height" value="0.0" />
-  <xacro:property name="camera_link_size" value="0.05" /> <!-- Size of square 'camera' box -->
+  <xacro:property name="camera_link_size" value="0.01" /> <!-- Size of square 'camera' box -->
   <!-- inertias for all links -->
   <xacro:macro name="default_inertial" params="mass">
@@ -58,5 +58,7 @@
     <parent link="base_link"/>
     <child link="base_yaw_link"/>
-    <origin xyz="0 0 0.126"/>
+    <origin
+      xyz="0 0 0.126"
+      rpy="0 0 0" />
     <axis xyz="0 0 1"/>
     <dynamics damping="1.0" friction="5.0"/>
@@ -66,13 +68,13 @@
   <link name="base_yaw_link">
     <visual>
-      <origin xyz="0 0 0" rpy="0 0 0" />
-      <geometry>
-        <mesh filename="package://dynamic_end_effector/meshes/assembly_base.stl" scale="0.001 0.001 0.001"/>
-      </geometry>
-    </visual>
-    <collision>
-      <origin xyz="0 0 0" rpy="0 0 0" />
-      <geometry>
-        <mesh filename="package://dynamic_end_effector/meshes/assembly_base.stl" scale="0.001 0.001 0.001"/>
+      <origin xyz="0 0 0" rpy="0 ${-pi/2} 0" />
+      <geometry>
+        <mesh filename="package://dynamic_end_effector/meshes/dynamixel_pro_frame.stl" scale="0.001 0.001 0.001"/>
+      </geometry>
+    </visual>
+    <collision>
+      <origin xyz="0 0 0" rpy="0 ${-pi/2} 0" />
+      <geometry>
+        <mesh filename="package://dynamic_end_effector/meshes/dynamixel_pro_frame.stl" scale="0.001 0.001 0.001"/>
       </geometry>
     </collision>
@@ -87,6 +89,6 @@
     <parent link="base_yaw_link"/>
     <child link="first_link"/>
-    <origin xyz="0 0 0.042"/>
-    <axis xyz="1 0 0"/>
+    <origin xyz="0 0 0.068"/>
+    <axis xyz="0 1 0"/>
     <dynamics damping="1.0" friction="1.0"/>
     <limit upper="2.0" lower="-2.0" effort="45" velocity="5"/>
@@ -95,13 +97,13 @@
   <link name="first_link">
     <visual>
-      <origin xyz="0 0 0" rpy="${pi/2.0} 0 0" />
-      <geometry>
-        <mesh filename="package://dynamic_end_effector/meshes/assembly_linkOne.stl" scale="0.001 0.001 0.001"/>
-      </geometry>
-    </visual>
-    <collision>
-      <origin xyz="0 0 0" rpy="${pi/2.0} 0 0" />
-      <geometry>
-        <mesh filename="package://dynamic_end_effector/meshes/assembly_linkOne.stl" scale="0.001 0.001 0.001"/>
+      <origin xyz="0 0 0" rpy="0 ${-pi/2} 0" />
+      <geometry>
+        <mesh filename="package://dynamic_end_effector/meshes/assembly_arm_1.stl" scale="0.001 0.001 0.001"/>
+      </geometry>
+    </visual>
+    <collision>
+      <origin xyz="0 0 0" rpy="0 ${-pi/2} 0" />
+      <geometry>
+        <mesh filename="package://dynamic_end_effector/meshes/assembly_arm_1.stl" scale="0.001 0.001 0.001"/>
       </geometry>
     </collision>
@@ -112,21 +114,21 @@
     <parent link="first_link"/>
     <child link="second_link"/>
-    <origin xyz="0 0 0.806"/>
-    <axis xyz="1 0 0"/>
-    <dynamics damping="1.0" friction="5.0"/>
-    <limit upper="${0.9*pi}" lower="${-0.9*pi}" effort="45" velocity="5"/>
+    <origin xyz="-0.033838 -0.006 0.430615"/>
+    <axis xyz="0 1 0"/>
+    <dynamics damping="1.0" friction="5.0"/>
+    <limit upper="${pi/4}" lower="${-pi}" effort="45" velocity="5"/>
   </joint>
   <xacro:transmission_block joint_name="first_link_to_second_link_joint"/>
   <link name="second_link">
     <visual>
-      <origin xyz="-0.033 0 0" rpy="${pi/2.0} -${pi/2.0} 0" />
-      <geometry>
-        <mesh filename="package://dynamic_end_effector/meshes/assembly_linkTwo.stl" scale="0.001 0.001 0.001"/>
-      </geometry>
-    </visual>
-    <collision>
-      <origin xyz="-0.033 0 0" rpy="${pi/2.0} -${pi/2.0} 0" />
-      <geometry>
-        <mesh filename="package://dynamic_end_effector/meshes/assembly_linkTwo.stl" scale="0.001 0.001 0.001"/>
+      <origin xyz="0 0 0" rpy="0 0 0" />
+      <geometry>
+        <mesh filename="package://dynamic_end_effector/meshes/assembly_arm_2.stl" scale="0.001 0.001 0.001"/>
+      </geometry>
+    </visual>
+    <collision>
+      <origin xyz="0 0 0" rpy="0 0 0" />
+      <geometry>
+        <mesh filename="package://dynamic_end_effector/meshes/assembly_arm_2.stl" scale="0.001 0.001 0.001"/>
       </geometry>
     </collision>
@@ -137,5 +139,5 @@
     <parent link="second_link"/>
     <child link="third_link"/>
-    <origin xyz="-0.06 0 0.61555"/>
+    <origin xyz="0.031 0.001 0.42"/>
     <axis xyz="0 0 1"/>
     <dynamics damping="1.0" friction="5.0"/>
@@ -145,13 +147,13 @@
   <link name="third_link">
     <visual>
-      <origin xyz="0 0 0" rpy="0 0 0" />
-      <geometry>
-        <mesh filename="package://dynamic_end_effector/meshes/assembly_linkThree.stl" scale="0.001 0.001 0.001"/>
-      </geometry>
-    </visual>
-    <collision>
-      <origin xyz="0 0 0" rpy="0 0 0" />
-      <geometry>
-        <mesh filename="package://dynamic_end_effector/meshes/assembly_linkThree.stl" scale="0.001 0.001 0.001"/>
+      <origin xyz="0 0 0" rpy="${pi/2} 0 0" />
+      <geometry>
+        <mesh filename="package://dynamic_end_effector/meshes/frame_mx108.stl" scale="0.001 0.001 0.001"/>
+      </geometry>
+    </visual>
+    <collision>
+      <origin xyz="0 0 0" rpy="${pi/2} 0 0" />
+      <geometry>
+        <mesh filename="package://dynamic_end_effector/meshes/frame_mx108.stl" scale="0.001 0.001 0.001"/>
       </geometry>
     </collision>
@@ -162,6 +164,6 @@
     <parent link="third_link"/>
     <child link="fourth_link"/>
-    <origin xyz="-0.025262 0 0.0383"/>
-    <axis xyz="1 0 0"/>
+    <origin xyz="0 0 0.037"/>
+    <axis xyz="0 1 0"/>
     <dynamics damping="1.0" friction="5.0"/>
     <limit upper="2.0" lower="-2.0" effort="45" velocity="5"/>
@@ -170,13 +172,13 @@
   <link name="fourth_link">
     <visual>
-      <origin xyz="0 0 0" rpy="${pi/2.0} 0 ${pi/2.0}" />
-      <geometry>
-        <mesh filename="package://dynamic_end_effector/meshes/assembly_linkFour.stl" scale="0.001 0.001 0.001"/>
-      </geometry>
-    </visual>
-    <collision>
-      <origin xyz="0 0 0" rpy="${pi/2.0} 0 ${pi/2.0}" />
-      <geometry>
-        <mesh filename="package://dynamic_end_effector/meshes/assembly_linkFour.stl" scale="0.001 0.001 0.001"/>
+      <origin xyz="0 0 0" rpy="${-pi/2} 0 ${pi/2}" />
+      <geometry>
+        <mesh filename="package://dynamic_end_effector/meshes/assembly_hand.stl" scale="0.001 0.001 0.001"/>
+      </geometry>
+    </visual>
+    <collision>
+      <origin xyz="0 0 0" rpy="${-pi/2} 0 ${pi/2}" />
+      <geometry>
+        <mesh filename="package://dynamic_end_effector/meshes/assembly_hand_simple.stl" scale="0.001 0.001 0.001"/>
       </geometry>
     </collision>
@@ -187,5 +189,5 @@
     <parent link="fourth_link"/>
     <child link="fifth_link"/>
-    <origin xyz="0.0278 0 0.09375"/>
+    <origin xyz="0 0 0.1198"/>
     <axis xyz="0 0 1"/>
     <dynamics damping="1.0" friction="5.0"/>
@@ -211,6 +213,6 @@
   <joint name="camera_joint" type="fixed">
     <!-- <axis xyz="0 1 0" /> -->
-    <origin xyz="0 0 ${camera_link_size/2 + 0.01}" rpy="0 ${-pi/2} 0"/>
-    <parent link="fifth_link"/>
+    <origin xyz="0 0.041 ${camera_link_size/2 + 0.114666}" rpy="0 ${-pi/2} 0"/>
+    <parent link="fourth_link"/>
     <child link="camera_link"/>
   </joint>

Commit message: added simple stl-files for collision checking

File: urdf/dynamic-ef.urdf.xacro (robot description, xacro)
@@ -1,4 +1,5 @@
 <?xml version="1.0"?>
-<robot name="dyn_ef_robot" xmlns:xacro="http://www.ros.org/wiki/xacro">
+<robot name="dyn_ef_robot"
+  xmlns:xacro="http://www.ros.org/wiki/xacro">
   <!-- Import all Gazebo-customization elements, including Gazebo colors -->
   <xacro:include filename="$(find dynamic_end_effector)/urdf/dynamic-ef.gazebo" />
@@ -12,5 +13,6 @@
   <!-- some properties for the urdf file -->
   <xacro:property name="height" value="0.0" />
-  <xacro:property name="camera_link_size" value="0.01" /> <!-- Size of square 'camera' box -->
+  <xacro:property name="camera_link_size" value="0.01" />
+  <!-- Size of square 'camera' box -->
   <!-- inertias for all links -->
   <xacro:macro name="default_inertial" params="mass">
@@ -49,5 +51,5 @@
       <origin xyz="0 0 0.09" rpy="${pi/2.0} 0 0" />
       <geometry>
-        <mesh filename="package://dynamic_end_effector/meshes/h54-200-s500-r.stl" scale="0.001 0.001 0.001"/>
+        <mesh filename="package://dynamic_end_effector/meshes/h54-200-s500-r_simple.stl" scale="0.001 0.001 0.001"/>
       </geometry>
     </collision>
@@ -58,7 +60,5 @@
     <parent link="base_link"/>
     <child link="base_yaw_link"/>
-    <origin
-      xyz="0 0 0.126"
-      rpy="0 0 0" />
+    <origin xyz="0 0 0.126" rpy="0 0 0" />
     <axis xyz="0 0 1"/>
     <dynamics damping="1.0" friction="5.0"/>
@@ -76,5 +76,5 @@
       <origin xyz="0 0 0" rpy="0 ${-pi/2} 0" />
       <geometry>
-        <mesh filename="package://dynamic_end_effector/meshes/dynamixel_pro_frame.stl" scale="0.001 0.001 0.001"/>
+        <mesh filename="package://dynamic_end_effector/meshes/dynamixel_pro_frame_simple.stl" scale="0.001 0.001 0.001"/>
       </geometry>
     </collision>
@@ -105,5 +105,5 @@
       <origin xyz="0 0 0" rpy="0 ${-pi/2} 0" />
       <geometry>
-        <mesh filename="package://dynamic_end_effector/meshes/assembly_arm_1.stl" scale="0.001 0.001 0.001"/>
+        <mesh filename="package://dynamic_end_effector/meshes/assembly_arm_1_simple.stl" scale="0.001 0.001 0.001"/>
       </geometry>
     </collision>
@@ -111,5 +111,5 @@
   </link>
   <joint name="first_link_to_second_link_joint" type="revolute">
-    <safety_controller k_position="100.0" k_velocity="40.0" soft_lower_limit="${-0.9*pi}" soft_upper_limit="${0.9*pi}"/>
+    <safety_controller k_position="100.0" k_velocity="40.0" soft_lower_limit="${-pi}" soft_upper_limit="${pi/4}"/>
     <parent link="first_link"/>
     <child link="second_link"/>
@@ -130,5 +130,5 @@
       <origin xyz="0 0 0" rpy="0 0 0" />
       <geometry>
-        <mesh filename="package://dynamic_end_effector/meshes/assembly_arm_2.stl" scale="0.001 0.001 0.001"/>
+        <mesh filename="package://dynamic_end_effector/meshes/assembly_arm_2_simple.stl" scale="0.001 0.001 0.001"/>
       </geometry>
     </collision>
@@ -161,5 +161,5 @@
   </link>
   <joint name="third_link_to_fourth_link_joint" type="revolute">
-    <safety_controller k_position="100.0" k_velocity="40.0" soft_lower_limit="-2.0" soft_upper_limit="2.0"/>
+    <safety_controller k_position="100.0" k_velocity="40.0" soft_lower_limit="-1.8" soft_upper_limit="1.8"/>
     <parent link="third_link"/>
     <child link="fourth_link"/>
@@ -167,5 +167,5 @@
     <axis xyz="0 1 0"/>
     <dynamics damping="1.0" friction="5.0"/>
-    <limit upper="2.0" lower="-2.0" effort="45" velocity="5"/>
+    <limit upper="1.8" lower="-1.8" effort="45" velocity="5"/>
   </joint>
   <xacro:transmission_block joint_name="third_link_to_fourth_link_joint"/>
@@ -219,16 +219,16 @@
   <!-- Camera -->
   <link name="camera_link">
-    <collision>
+    <visual>
       <origin xyz="0 0 0" rpy="0 0 0"/>
       <geometry>
         <box size="${camera_link_size} ${camera_link_size} ${camera_link_size}"/>
       </geometry>
-    </collision>
-    <visual>
+    </visual>
+    <collision>
       <origin xyz="0 0 0" rpy="0 0 0"/>
       <geometry>
         <box size="${camera_link_size} ${camera_link_size} ${camera_link_size}"/>
       </geometry>
-    </visual>
+    </collision>
     <inertial>
       <mass value="1e-5" />

Commit message: edited urdf to represent the real robot

File: urdf/dynamic-ef.urdf.xacro (robot description, xacro)
@@ -68,13 +68,13 @@
   <link name="base_yaw_link">
     <visual>
-      <origin xyz="0 0 0" rpy="0 ${-pi/2} 0" />
-      <geometry>
-        <mesh filename="package://dynamic_end_effector/meshes/dynamixel_pro_frame.stl" scale="0.001 0.001 0.001"/>
-      </geometry>
-    </visual>
-    <collision>
-      <origin xyz="0 0 0" rpy="0 ${-pi/2} 0" />
-      <geometry>
-        <mesh filename="package://dynamic_end_effector/meshes/dynamixel_pro_frame_simple.stl" scale="0.001 0.001 0.001"/>
+      <origin xyz="0 0 0" rpy="0 ${-pi} 0" />
+      <geometry>
+        <mesh filename="package://dynamic_end_effector/meshes/assembly_link2.stl" scale="0.001 0.001 0.001"/>
+      </geometry>
+    </visual>
+    <collision>
+      <origin xyz="0 0 0" rpy="0 ${-pi} 0" />
+      <geometry>
+        <mesh filename="package://dynamic_end_effector/meshes/assembly_link2_simple.stl" scale="0.001 0.001 0.001"/>
       </geometry>
     </collision>
@@ -89,5 +89,5 @@
     <parent link="base_yaw_link"/>
     <child link="first_link"/>
-    <origin xyz="0 0 0.068"/>
+    <origin xyz="0 0 0.0392"/>
     <axis xyz="0 1 0"/>
     <dynamics damping="1.0" friction="1.0"/>
@@ -97,5 +97,5 @@
   <link name="first_link">
     <visual>
-      <origin xyz="0 0 0" rpy="0 ${-pi/2} 0" />
+      <origin xyz="0 0 0" rpy="0 0 ${-pi/2}" />
       <geometry>
         <mesh filename="package://dynamic_end_effector/meshes/assembly_arm_1.stl" scale="0.001 0.001 0.001"/>
@@ -103,5 +103,5 @@
     </visual>
     <collision>
-      <origin xyz="0 0 0" rpy="0 ${-pi/2} 0" />
+      <origin xyz="0 0 0" rpy="0 0 ${-pi/2}" />
       <geometry>
         <mesh filename="package://dynamic_end_effector/meshes/assembly_arm_1_simple.stl" scale="0.001 0.001 0.001"/>
@@ -111,16 +111,16 @@
   </link>
   <joint name="first_link_to_second_link_joint" type="revolute">
-    <safety_controller k_position="100.0" k_velocity="40.0" soft_lower_limit="${-pi}" soft_upper_limit="${pi/4}"/>
+    <safety_controller k_position="100.0" k_velocity="40.0" soft_lower_limit="${-pi/4}" soft_upper_limit="${pi}"/>
     <parent link="first_link"/>
     <child link="second_link"/>
-    <origin xyz="-0.033838 -0.006 0.430615"/>
+    <origin xyz="0.034613 0.00625 0.457247"/>
     <axis xyz="0 1 0"/>
     <dynamics damping="1.0" friction="5.0"/>
-    <limit upper="${pi/4}" lower="${-pi}" effort="45" velocity="5"/>
+    <limit lower="${-pi/4}" upper="${pi}" effort="45" velocity="5"/>
   </joint>
   <xacro:transmission_block joint_name="first_link_to_second_link_joint"/>
   <link name="second_link">
     <visual>
-      <origin xyz="0 0 0" rpy="0 0 0" />
+      <origin xyz="0 0 0" rpy="0 0 ${pi/2}" />
       <geometry>
         <mesh filename="package://dynamic_end_effector/meshes/assembly_arm_2.stl" scale="0.001 0.001 0.001"/>
@@ -128,5 +128,5 @@
     </visual>
     <collision>
-      <origin xyz="0 0 0" rpy="0 0 0" />
+      <origin xyz="0 0 0" rpy="0 0 ${pi/2}" />
       <geometry>
         <mesh filename="package://dynamic_end_effector/meshes/assembly_arm_2_simple.stl" scale="0.001 0.001 0.001"/>
@@ -139,5 +139,5 @@
     <parent link="second_link"/>
     <child link="third_link"/>
-    <origin xyz="0.031 0.001 0.42"/>
+    <origin xyz="-0.031 -0.001 0.422"/>
     <axis xyz="0 0 1"/>
     <dynamics damping="1.0" friction="5.0"/>
@@ -155,5 +155,5 @@
       <origin xyz="0 0 0" rpy="${pi/2} 0 0" />
       <geometry>
-        <mesh filename="package://dynamic_end_effector/meshes/frame_mx108.stl" scale="0.001 0.001 0.001"/>
+        <mesh filename="package://dynamic_end_effector/meshes/frame_mx108_simple.stl" scale="0.001 0.001 0.001"/>
       </geometry>
     </collision>
@@ -189,5 +189,5 @@
     <parent link="fourth_link"/>
     <child link="fifth_link"/>
-    <origin xyz="0 0 0.1198"/>
+    <origin xyz="0 0.0005 0.1233"/>
     <axis xyz="0 0 1"/>
     <dynamics damping="1.0" friction="5.0"/>
@@ -197,13 +197,13 @@
   <link name="fifth_link">
     <visual>
-      <origin xyz="0 0 0" rpy="${pi/2.0} 0 0" />
-      <geometry>
-        <mesh filename="package://dynamic_end_effector/meshes/assembly_linkFive.stl" scale="0.001 0.001 0.001"/>
-      </geometry>
-    </visual>
-    <collision>
-      <origin xyz="0 0 0" rpy="${pi/2.0} 0 0" />
-      <geometry>
-        <mesh filename="package://dynamic_end_effector/meshes/assembly_linkFive.stl" scale="0.001 0.001 0.001"/>
+      <origin xyz="0.004143 -0.006953 0.004" rpy="0 0 0" />
+      <geometry>
+        <mesh filename="package://dynamic_end_effector/meshes/Pointing_Finger2.stl" scale="0.001 0.001 0.001"/>
+      </geometry>
+    </visual>
+    <collision>
+      <origin xyz="0.004143 -0.006953 0.004" rpy="0 0 0" />
+      <geometry>
+        <mesh filename="package://dynamic_end_effector/meshes/Pointing_Finger2_simple.stl" scale="0.001 0.001 0.001"/>
       </geometry>
     </collision>

Commit message: adjusting joint limits

File: urdf/dynamic-ef.urdf.xacro (robot description, xacro)
@@ -22,13 +22,13 @@
     </inertial>
   </xacro:macro>
-  <!-- interface between moveit and gazebo controllers -->
+  <!-- interface between moveit and real robot controllers -->
   <xacro:macro name="transmission_block" params="joint_name">
     <transmission name="trans_${joint_name}">
       <type>transmission_interface/SimpleTransmission</type>
       <joint name="${joint_name}">
-        <hardwareInterface>hardware_interface/PositionJointInterface</hardwareInterface>
+        <hardwareInterface>hardware_interface/VelocityJointInterface</hardwareInterface>
       </joint>
       <actuator name="motor_${joint_name}">
-        <hardwareInterface>hardware_interface/PositionJointInterface</hardwareInterface>
+        <hardwareInterface>hardware_interface/VelocityJointInterface</hardwareInterface>
         <mechanicalReduction>1</mechanicalReduction>
       </actuator>
@@ -57,5 +57,5 @@
   </link>
   <joint name="base_link_to_base_yaw_link_joint" type="revolute">
-    <safety_controller k_position="100.0" k_velocity="40.0" soft_lower_limit="${-pi}" soft_upper_limit="${pi}"/>
+    <!-- <safety_controller k_position="100.0" k_velocity="40.0" soft_lower_limit="${-2.0}" soft_upper_limit="${2.0}"/> -->
     <parent link="base_link"/>
     <child link="base_yaw_link"/>
@@ -63,5 +63,5 @@
     <axis xyz="0 0 1"/>
     <dynamics damping="1.0" friction="5.0"/>
-    <limit upper="${pi}" lower="${-pi}" effort="45" velocity="5"/>
+    <limit upper="${2.0}" lower="${-2.0}" effort="45" velocity="5"/>
   </joint>
   <xacro:transmission_block joint_name="base_link_to_base_yaw_link_joint"/>
@@ -86,5 +86,5 @@
   </link>
   <joint name="base_yaw_link_to_first_link_joint" type="revolute">
-    <safety_controller k_position="100.0" k_velocity="40.0" soft_lower_limit="-2.0" soft_upper_limit="2.0"/>
+    <!-- <safety_controller k_position="100.0" k_velocity="40.0" soft_lower_limit="-2.0" soft_upper_limit="2.0"/> -->
     <parent link="base_yaw_link"/>
     <child link="first_link"/>
@@ -111,5 +111,5 @@
   </link>
   <joint name="first_link_to_second_link_joint" type="revolute">
-    <safety_controller k_position="100.0" k_velocity="40.0" soft_lower_limit="${-pi/4}" soft_upper_limit="${pi}"/>
+    <!-- <safety_controller k_position="100.0" k_velocity="40.0" soft_lower_limit="${-pi/4}" soft_upper_limit="${pi}"/> -->
     <parent link="first_link"/>
     <child link="second_link"/>
@@ -135,6 +135,6 @@
     <xacro:default_inertial mass="1"/>
   </link>
-  <joint name="second_link_to_third_link_joint" type="continuous">
-    <safety_controller k_position="100.0" k_velocity="40.0" soft_lower_limit="${-pi}" soft_upper_limit="${pi}"/>
+  <joint name="second_link_to_third_link_joint" type="revolute">
+    <!-- <safety_controller k_position="100.0" k_velocity="40.0" soft_lower_limit="${-pi/2}" soft_upper_limit="${3*pi/2}"/> -->
     <parent link="second_link"/>
     <child link="third_link"/>
@@ -142,5 +142,5 @@
     <axis xyz="0 0 1"/>
     <dynamics damping="1.0" friction="5.0"/>
-    <limit upper="${pi}" lower="${-pi}" effort="45" velocity="5"/>
+    <limit upper="${3*pi/2}" lower="${-pi/2}" effort="45" velocity="5"/>
   </joint>
   <xacro:transmission_block joint_name="second_link_to_third_link_joint"/>
@@ -161,5 +161,5 @@
   </link>
   <joint name="third_link_to_fourth_link_joint" type="revolute">
-    <safety_controller k_position="100.0" k_velocity="40.0" soft_lower_limit="-1.8" soft_upper_limit="1.8"/>
+    <!-- <safety_controller k_position="100.0" k_velocity="40.0" soft_lower_limit="-1.8" soft_upper_limit="1.8"/> -->
     <parent link="third_link"/>
     <child link="fourth_link"/>
@@ -186,5 +186,5 @@
   </link>
   <joint name="fourth_link_to_fifth_link_joint" type="revolute">
-    <safety_controller k_position="100.0" k_velocity="40.0" soft_lower_limit="${-pi}" soft_upper_limit="${pi}"/>
+    <!-- <safety_controller k_position="100.0" k_velocity="40.0" soft_lower_limit="${-pi}" soft_upper_limit="${pi}"/> -->
     <parent link="fourth_link"/>
     <child link="fifth_link"/>
@@ -192,5 +192,5 @@
     <axis xyz="0 0 1"/>
     <dynamics damping="1.0" friction="5.0"/>
-    <limit upper="${pi}" lower="${-pi}" effort="45" velocity="5"/>
+    <limit upper="${pi*2}" lower="${-pi*2}" effort="45" velocity="5"/>
   </joint>
   <xacro:transmission_block joint_name="fourth_link_to_fifth_link_joint"/>

Commit message: clean up. remove unnecessary files

File: urdf/dynamic-ef.urdf.xacro (robot description, xacro)
@@ -13,6 +13,5 @@
   <!-- some properties for the urdf file -->
   <xacro:property name="height" value="0.0" />
-  <xacro:property name="camera_link_size" value="0.01" />
-  <!-- Size of square 'camera' box -->
+  <xacro:property name="camera_link_size" value="0.01" /> <!-- Size of square 'camera' box -->
   <!-- inertias for all links -->
   <xacro:macro name="default_inertial" params="mass">

Commit message: change controllers to velocityController

File: urdf/dynamic-ef.urdf.xacro (robot description, xacro)
@@ -212,5 +212,5 @@
   <joint name="camera_joint" type="fixed">
     <!-- <axis xyz="0 1 0" /> -->
-    <origin xyz="0 0.041 ${camera_link_size/2 + 0.114666}" rpy="0 ${-pi/2} 0"/>
+    <origin xyz="0 0.041 ${camera_link_size/2 + 0.099666}" rpy="0 ${-pi/2} 0"/>
     <parent link="fourth_link"/>
     <child link="camera_link"/>

Commit message: corrected camera orientation, changed gazebo parameters for realtime assurance

File: urdf/dynamic-ef.urdf.xacro (robot description, xacro)
@@ -212,5 +212,5 @@
   <joint name="camera_joint" type="fixed">
     <!-- <axis xyz="0 1 0" /> -->
-    <origin xyz="0 0.041 ${camera_link_size/2 + 0.099666}" rpy="0 ${-pi/2} 0"/>
+    <origin xyz="0 0.041 ${camera_link_size/2 + 0.099666}" rpy="0 ${-pi/2} ${-pi/2}"/>
     <parent link="fourth_link"/>
     <child link="camera_link"/>
